File: Schematics/MinisumoV2/MinisumoV2.kicad_pcb (KiCad board)
At the start: 2 copper layers, 80 x 67 mm, 85 parts, among them J1 SWD_CONNECTOR, J10 LINE_RIGHT, J11 LINE_LEFT, J2 BATT, J3 MOTOR_L_1, J4 MOTOR_L_2, J5 MOTOR_R_1, J6 MOTOR_R_2, J7 TOF_RIGHT, J8 TOF_CENTER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

Commit message: HW: Minisumo PCB v1
Parts:
- removed J7: TOF_RIGHT, Connector_JST:JST_PH_B4B-PH-K_1x04_P2.00mm_Vertical
- removed J8: TOF_CENTER, Connector_JST:JST_PH_B4B-PH-K_1x04_P2.00mm_Vertical
- removed J9: TOF_LEFT, Connector_JST:JST_PH_B4B-PH-K_1x04_P2.00mm_Vertical
- added G***: LOGO, LOGO, B.Cu at (187.0, 134.8)
- added G***: LOGO, LOGO, B.Cu at (166.1, 126.4)
- added J12: SHARP_CENTER, Connector_PinHeader_1.27mm:PinHeader_2x04_P1.27mm_Vertical, F.Cu at (186.0, 97.6)
- added J13: SHARP_LEFT, Connector_PinHeader_1.27mm:PinHeader_2x04_P1.27mm_Vertical, F.Cu at (175.8, 96.6)
- added J14: SHARP_RIGHT, Connector_PinHeader_1.27mm:PinHeader_2x04_P1.27mm_Vertical, F.Cu at (198.3, 97.6)
- added kibuzzard-69A732F2: G***, kibuzzard-69A732F2, F.Cu at (193.3, 108.8)
- added kibuzzard-69A73765: G***, kibuzzard-69A73765, B.Cu at (209.6, 99.6)
- added kibuzzard-69A73775: G***, kibuzzard-69A73775, B.Cu at (164.9, 97.6)
- added kibuzzard-69A73CC0: G***, kibuzzard-69A73CC0, F.Cu at (146.9, 113.9)
Connections:
- U1 pad 16: unconnected-(U1-PA6-Pad16) -> /SHARP_C_ANALOG
- U1 pad 17: /MOTOR_ENABLE -> /SHARP_L_ANALOG
- U1 pad 18: unconnected-(U1-PB0-Pad18) -> /SHARP_R_ANALOG
- U1 pad 21: /TOF_RIGHT_SCL -> /SHARP_L_SCL
- U1 pad 25: /TOF_RIGHT_SDA -> /SHARP_L_SDA
- U1 pad 26: unconnected-(U1-PB13-Pad26) -> /MOTOR_ENABLE
- U1 pad 29: /TOF_LEFT_SCL -> /SHARP_R_SCL
- U1 pad 40: /TOF_LEFT_SDA -> /SHARP_R_SDA
- U1 pad 42: /TOF_CENTER_SCL -> /SHARP_C_SCL
- U1 pad 43: /TOF_CENTER_SDA -> /SHARP_C_SDA
Routing:
- net /SHARP_R_SCL: track 0.00 -> 34.2 mm, vias 0 -> 3
- net /TOF_LEFT_SCL: track 32.2 -> 0.00 mm, vias 1 -> 0
- net /SHARP_R_ANALOG: track 0.00 -> 29.0 mm, vias 0 -> 2
- net /SHARP_R_SDA: track 0.00 -> 26.5 mm, vias 0 -> 2
- net /TOF_LEFT_SDA: track 26.1 -> 0.00 mm, vias 1 -> 0
- net +3V3: track 177.6 -> 201.0 mm
- net /SHARP_L_SDA: track 0.00 -> 22.0 mm, vias 0 -> 1
- net /SHARP_L_SCL: track 0.00 -> 21.9 mm, vias 0 -> 1
- net /SHARP_C_SCL: track 0.00 -> 21.6 mm, vias 0 -> 2
- net /TOF_RIGHT_SDA: track 20.8 -> 0.00 mm, vias 1 -> 0
- net /SHARP_C_ANALOG: track 0.00 -> 19.5 mm, vias 0 -> 1
- net /TOF_CENTER_SCL: track 16.6 -> 0.00 mm, vias 1 -> 0
- net /SHARP_L_ANALOG: track 0.00 -> 15.8 mm, vias 0 -> 1
- net /TOF_RIGHT_SCL: track 15.6 -> 0.00 mm, vias 1 -> 0
- net /SHARP_C_SDA: track 0.00 -> 14.6 mm, vias 0 -> 2
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Other:
- outline, holes or cut-outs redrawn
