File: Schematics/MinisumoV2/MinisumoV2.kicad_pcb (KiCad board)
At the start: 2 copper layers, 80 x 67 mm, 91 parts, among them J1 SWD_CONNECTOR, J10 LINE_RIGHT, J11 LINE_LEFT, J12 SHARP_CENTER, J13 SHARP_LEFT, J14 SHARP_RIGHT, J2 BATT, J3 MOTOR_L_1, J4 MOTOR_L_2, J5 MOTOR_R_1, J6 MOTOR_R_2, Q4 IRLML2502, SW1 SW_DIP_x04, U1 STM32H523CCTx, U2 TPS563201, U3 AMS1117-3.3, U4 LM358, U5 MP6551, U6 MP6551, U7 IRM-56384

Commit message: Update PCB
Parts:
- removed the G*** at (193.1, 123.0)
- removed J12: SHARP_CENTER, Connector_PinHeader_1.27mm:PinHeader_2x04_P1.27mm_Vertical
- removed J13: SHARP_LEFT, Connector_PinHeader_1.27mm:PinHeader_2x04_P1.27mm_Vertical
- removed J14: SHARP_RIGHT, Connector_PinHeader_1.27mm:PinHeader_2x04_P1.27mm_Vertical
- removed the REF** at (159.9, 127.8)
- added J15: SHARP_LEFT, Connector_PinHeader_2.00mm:PinHeader_1x03_P2.00mm_Vertical, F.Cu at (175.1, 95.9)
- added J7: UART_DBG, Connector_PinHeader_2.54mm:PinHeader_1x04_P2.54mm_Vertical, F.Cu at (211.1, 110.7)
- added J8: SHARP_RIGHT, Connector_PinHeader_2.00mm:PinHeader_1x03_P2.00mm_Vertical, F.Cu at (197.6, 95.9)
- added J9: SHARP_CENTER, Connector_PinHeader_2.00mm:PinHeader_1x03_P2.00mm_Vertical, F.Cu at (185.9, 95.9)
- added JP1: BYPASS, Jumper:SolderJumper-2_P1.3mm_Open_RoundedPad1.0x1.5mm, F.Cu at (171.4, 118.1)
- added REF**: OSHW-Logo2_7.3x6mm_SilkScreen, Symbol:OSHW-Logo2_7.3x6mm_SilkScreen, F.Cu at (157.5, 121.4)
- added REF**: KiCad-Logo2_5mm_SilkScreen, Symbol:KiCad-Logo2_5mm_SilkScreen, F.Cu at (192.8, 122.2)
- added kibuzzard-69A73775: G***, kibuzzard-69A73775, B.Cu at (177.5, 98.6)
- added kibuzzard-69A73775: G***, kibuzzard-69A73775, B.Cu at (199.6, 98.6)
- added kibuzzard-69A73775: G***, kibuzzard-69A73775, B.Cu at (188.0, 98.6)
- added kibuzzard-6A21495C: G***, kibuzzard-6A21495C, F.Cu at (213.9, 107.2)
- J10, J11: footprint Connector_PinHeader_2.54mm:PinHeader_1x03_P2.54mm_Vertical -> Connector_PinHeader_2.00mm:PinHeader_1x03_P2.00mm_Vertical
Connections:
- U1 pad 19: unconnected-(U1-PB1-Pad19) -> /IR_STARTSTOP
- U1 pad 21: /SHARP_L_SCL -> unconnected-(U1-PB10-Pad21)
- U1 pad 25: /SHARP_L_SDA -> unconnected-(U1-PB12-Pad25)
- U1 pad 29: /SHARP_R_SCL -> /TOF_LEFT_SCL
- U1 pad 40: /SHARP_R_SDA -> unconnected-(U1-PB4(NJTRST)-Pad40)
- U1 pad 41: unconnected-(U1-PB5-Pad41) -> /UART_RX
- U1 pad 42: /SHARP_C_SCL -> /UART_TX
- U1 pad 43: /SHARP_C_SDA -> unconnected-(U1-PB7-Pad43)
Routing:
- net /UART_RX: track 0.00 -> 37.0 mm, vias 0 -> 1
- net /UART_TX: track 0.00 -> 35.7 mm, vias 0 -> 1
- net /SHARP_R_SCL: track 34.2 -> 0.00 mm, vias 3 -> 0
- net /SHARP_R_SDA: track 26.5 -> 0.00 mm, vias 2 -> 0
- net /SHARP_L_SDA: track 22.0 -> 0.00 mm, vias 1 -> 0
- net /SHARP_L_SCL: track 21.9 -> 0.00 mm, vias 1 -> 0
- net /SHARP_C_SCL: track 21.6 -> 0.00 mm, vias 2 -> 0
- net /SHARP_C_SDA: track 14.6 -> 0.00 mm, vias 2 -> 0
- net /IR_STARTSTOP: track 0.00 -> 14.2 mm, vias 0 -> 2
- net /SHARP_C_ANALOG: track 19.5 -> 33.1 mm, vias 1 -> 2
- net +3V3: track 201.0 -> 190.5 mm
- net /SHARP_R_ANALOG: track 29.0 -> 20.7 mm, vias 2 -> 1
- net GND: track 37.9 -> 32.4 mm, vias 279 -> 277
- net /LEDS_WS: track 13.9 -> 16.8 mm
- net Net-(D4-DIN): track 4.76 -> 7.54 mm
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Other:
- board text added: "Creado por @LaboratorioGluon"
- board text added: "Version 1.1"
