File: Schematics/MinisumoV2/MinisumoV2.kicad_sch (KiCad schematic)
At the start: 40 parts, among them J1 SWD_CONNECTOR, J10 LINE_RIGHT, J11 LINE_LEFT, J7 TOF_RIGHT, J8 TOF_CENTER, J9 TOF_LEFT, Q4 IRLML2502, SW1 SW_DIP_x04, U1 STM32H523CCTx, U7 IRM-56384

Commit message: HW: Minisumo PCB v1
Parts:
- removed J7: TOF_RIGHT, Connector_JST:JST_PH_B4B-PH-K_1x04_P2.00mm_Vertical, symbol Connector_Generic:Conn_01x04
- removed J8: TOF_CENTER, Connector_JST:JST_PH_B4B-PH-K_1x04_P2.00mm_Vertical, symbol Connector_Generic:Conn_01x04
- removed J9: TOF_LEFT, Connector_JST:JST_PH_B4B-PH-K_1x04_P2.00mm_Vertical, symbol Connector_Generic:Conn_01x04
- added J12: SHARP_CENTER, Connector_PinHeader_1.27mm:PinHeader_2x04_P1.27mm_Vertical, symbol Connector_Generic:Conn_01x07
- added J13: SHARP_LEFT, Connector_PinHeader_1.27mm:PinHeader_2x04_P1.27mm_Vertical, symbol Connector_Generic:Conn_01x07
- added J14: SHARP_RIGHT, Connector_PinHeader_1.27mm:PinHeader_2x04_P1.27mm_Vertical, symbol Connector_Generic:Conn_01x07
Connections:
- net +3V3: now also J12.1 (Pin_1), J12.4 (Pin_4), J12.5 (Pin_5), J13.1 (Pin_1), J13.4 (Pin_4), J13.5 (Pin_5), J14.1 (Pin_1), J14.4 (Pin_4), J14.5 (Pin_5)
- net GND: now also J12.3 (Pin_3), J13.3 (Pin_3), J14.3 (Pin_3)
- net MOTOR_ENABLE: now also U1.26 (PB13); no longer U1.17 (PA7)
- net SHARP_C_ANALOG: now reaches U1.16 (PA6)
- net SHARP_C_ANALOG: now also J12.2 (Pin_2)
- net SHARP_R_ANALOG: now reaches U1.18 (PB0)
- net SHARP_R_ANALOG: now also J14.2 (Pin_2)
- net TOF_CENTER_SCL renamed SHARP_C_SCL
- net SHARP_C_SCL: now also J12.6 (Pin_6)
- net TOF_CENTER_SDA renamed SHARP_C_SDA
- net SHARP_C_SDA: now also J12.7 (Pin_7)
- net TOF_LEFT_SCL renamed SHARP_L_SCL
- net SHARP_L_SCL: now also J13.6 (Pin_6)
- net TOF_LEFT_SDA renamed SHARP_L_SDA
- net SHARP_L_SDA: now also J13.7 (Pin_7)
- net TOF_RIGHT_SCL renamed SHARP_R_SCL
- net SHARP_R_SCL: now also J14.6 (Pin_6)
- net TOF_RIGHT_SDA renamed SHARP_R_SDA
- net SHARP_R_SDA: now also J14.7 (Pin_7)
- new net SHARP_L_ANALOG: J13.2 (Pin_2), U1.17 (PA7)
- no-connect marks 16 -> 13
Changed lines of the file:
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@@
 (kicad_sch
-	(version 20250114)
+	(version 20260306)
 	(generator "eeschema")
-	(generator_version "9.0")
+	(generator_version "10.0")
 	(paper "A4")
