File: Schematics/MinisumoV2/MinisumoV2.kicad_sch (KiCad schematic)
At the start: 40 parts, among them J1 SWD_CONNECTOR, J10 LINE_RIGHT, J11 LINE_LEFT, J12 SHARP_CENTER, J13 SHARP_LEFT, J14 SHARP_RIGHT, Q4 IRLML2502, SW1 SW_DIP_x04, U1 STM32H523CCTx, U7 IRM-56384

Commit message: Update PCB
Parts:
- removed J12: SHARP_CENTER, Connector_PinHeader_1.27mm:PinHeader_2x04_P1.27mm_Vertical, symbol Connector_Generic:Conn_01x07
- removed J13: SHARP_LEFT, Connector_PinHeader_1.27mm:PinHeader_2x04_P1.27mm_Vertical, symbol Connector_Generic:Conn_01x07
- removed J14: SHARP_RIGHT, Connector_PinHeader_1.27mm:PinHeader_2x04_P1.27mm_Vertical, symbol Connector_Generic:Conn_01x07
- added J15: SHARP_LEFT, Connector_PinHeader_2.00mm:PinHeader_1x03_P2.00mm_Vertical, symbol Connector_Generic:Conn_01x03
- added J7: UART_DBG, Connector_PinHeader_2.54mm:PinHeader_1x04_P2.54mm_Vertical, symbol Connector_Generic:Conn_01x04
- added J8: SHARP_RIGHT, Connector_PinHeader_2.00mm:PinHeader_1x03_P2.00mm_Vertical, symbol Connector_Generic:Conn_01x03
- added J9: SHARP_CENTER, Connector_PinHeader_2.00mm:PinHeader_1x03_P2.00mm_Vertical, symbol Connector_Generic:Conn_01x03
- added JP1: BYPASS, Jumper:SolderJumper-2_P1.3mm_Open_RoundedPad1.0x1.5mm, symbol Jumper:SolderJumper_2_Open
- J10, J11: footprint Connector_PinHeader_2.54mm:PinHeader_1x03_P2.54mm_Vertical -> Connector_PinHeader_2.00mm:PinHeader_1x03_P2.00mm_Vertical
Connections:
- net +3V3: now also J15.1 (Pin_1), J7.3 (Pin_3), J8.1 (Pin_1), J9.1 (Pin_1)
- net GND: now also J15.3 (Pin_3), J7.4 (Pin_4), J8.3 (Pin_3), J9.3 (Pin_3)
- net IR_STARTSTOP: now also U1.19 (PB1)
- net LEDS_WS: now also JP1.1 (A)
- net SHARP_C_ANALOG: now also J8.2 (Pin_2)
- net SHARP_L_ANALOG: now also J15.2 (Pin_2)
- net SHARP_R_ANALOG: now also J9.2 (Pin_2)
- net at D4.4 (DIN), R26.1: now also JP1.2 (B)
- net UART_RX: now reaches U1.41 (PB5)
- net UART_RX: now also J7.1 (Pin_1)
- net SHARP_C_SCL renamed UART_TX
- net UART_TX: now also J7.2 (Pin_2)
- net SHARP_C_SDA: no longer names the net of U1.43 (PB7)
- net SHARP_L_SCL renamed TOF_LEFT_SCL
- net SHARP_L_SDA: no longer names the net of U1.40 (PB4(NJTRST))
- net SHARP_R_SCL: no longer names the net of U1.21 (PB10)
- net SHARP_R_SDA: no longer names the net of U1.25 (PB12)
- no-connect marks 13 -> 15
Other:
- moved on the sheet: R27
